File: kicad/ttp5_mqtt/ttp5_mqtt.kicad_pcb (KiCad board)
At the start: 2 copper layers, 2 parts, among them U1 TSR_1-2433

Commit message: add sources
Parts:
- added C1: 22n, Resistor_SMD:R_0603_1608Metric_Pad0.98x0.95mm_HandSolder, B.Cu at (165.7, 68.8)
- added H1: MountingHole, MountingHole:MountingHole_6.5mm, F.Cu at (169.2, 97.2)
- added J1: Conn_water, Connector_PinHeader_2.54mm:PinHeader_2x01_P2.54mm_Vertical, F.Cu at (178.0, 99.8)
- added J2: Conn_pump, Connector_PinHeader_2.54mm:PinHeader_2x01_P2.54mm_Vertical, F.Cu at (173.2, 67.8)
- added J3: Conn_Power, Connector_Molex:Molex_KK-396_A-41791-0002_1x02_P3.96mm_Vertical, F.Cu at (164.8, 62.2)
- added J4: Conn_waterlevel, Connector_PinHeader_2.54mm:PinHeader_2x01_P2.54mm_Vertical, F.Cu at (180.8, 87.8)
- added J5: Conn_01x04, Connector_PinHeader_2.54mm:PinHeader_1x04_P2.54mm_Vertical, F.Cu at (157.0, 100.5)
- added K1: FINDER-34.51, Relay_THT:Relay_SPDT_Finder_34.51_Vertical, F.Cu at (161.0, 81.2)
- added Q1: IRLZ44N, PCM_Package_TO_SOT_THT_AKL:TO-220-3_Vertical_GDS, F.Cu at (179.0, 68.2)
- added Q2: IRLZ44N, PCM_Package_TO_SOT_THT_AKL:TO-220-3_Vertical_GDS, F.Cu at (179.0, 57.7)
- added R1: 47k, Resistor_SMD:R_0201_0603Metric_Pad0.64x0.40mm_HandSolder, B.Cu at (176.9, 119.2)
- added R2: 47k, Resistor_SMD:R_0201_0603Metric_Pad0.64x0.40mm_HandSolder, B.Cu at (176.9, 115.6)
- added R3: 47k, Resistor_SMD:R_0201_0603Metric_Pad0.64x0.40mm_HandSolder, B.Cu at (176.9, 112.0)
- U1: value TSR_1-2433 -> TSR_1-2450
- moved U1 33.9 mm to (161.7, 73.0)
- moved ESP32C6 26.0 mm to (159.6, 106.3), turned to -90 degrees
Connections:
- ESP32C6 pad 1: unconnected-(ESP32C6-5V-Pad1) -> +5V
- ESP32C6 pad 3: Net-(ESP32C6-3.3V) -> +3.3V
- ESP32C6 pad 4: unconnected-(ESP32C6-GP0-Pad4) -> Net-(ESP32C6-GP0)
- ESP32C6 pad 5: unconnected-(ESP32C6-GP1-Pad5) -> Net-(ESP32C6-GP1)
- ESP32C6 pad 6: unconnected-(ESP32C6-GP2-Pad6) -> /waterlevel_in
- ESP32C6 pad 7: unconnected-(ESP32C6-GP3-Pad7) -> /humidity_scl_i2c
- ESP32C6 pad 8: unconnected-(ESP32C6-GP4-Pad8) -> /humidity_sda_i2c
- U1 pad 1: unconnected-(U1-Vin-Pad1) -> +9V
- U1 pad 2: unconnected-(U1-GND-Pad2) -> GND
- U1 pad 3: Net-(ESP32C6-3.3V) -> +5V
Routing:
- net GND: track 0.00 -> 115.5 mm, vias 0 -> 1
- net Net-(ESP32C6-GP1): track 0.00 -> 62.3 mm, vias 0 -> 1
- net Net-(ESP32C6-GP0): track 0.00 -> 54.9 mm, vias 0 -> 1
- net +3.3V: track 0.00 -> 49.5 mm
- net +5V: track 0.00 -> 45.4 mm
- net /waterlevel_in: track 0.00 -> 39.1 mm, vias 0 -> 1
- net +9V: track 0.00 -> 33.6 mm
- net Net-(Q1-D): track 0.00 -> 26.3 mm
- net Net-(J1-Pin_1): track 0.00 -> 19.3 mm
- net Net-(J1-Pin_2): track 0.00 -> 17.7 mm
- net /humidity_scl_i2c: track 0.00 -> 17.4 mm
- net /humidity_sda_i2c: track 0.00 -> 13.8 mm
- net Net-(J2-Pin_2): track 0.00 -> 8.54 mm
Other:
- board outline added: 30 x 74.5 mm
- copper layers 2 -> 4
