File: kicad/ttp5_mqtt/ttp5_mqtt.kicad_sch (KiCad schematic)
At the start: 2 parts, among them U1 TSR_1-2433

Commit message: add sources
Parts:
- added C1: 22n, Resistor_SMD:R_0603_1608Metric_Pad0.98x0.95mm_HandSolder, symbol Device:C_Small
- added H1: MountingHole, MountingHole:MountingHole_6.5mm, symbol Mechanical:MountingHole
- added J1: Conn_water, Connector_PinHeader_2.54mm:PinHeader_2x01_P2.54mm_Vertical, symbol Connector_Generic:Conn_02x01
- added J2: Conn_pump, Connector_PinHeader_2.54mm:PinHeader_2x01_P2.54mm_Vertical, symbol Connector_Generic:Conn_02x01
- added J3: Conn_Power, Connector_Molex:Molex_KK-396_A-41791-0002_1x02_P3.96mm_Vertical, symbol Connector_Generic:Conn_02x01
- added J4: Conn_waterlevel, Connector_PinHeader_2.54mm:PinHeader_2x01_P2.54mm_Vertical, symbol Connector_Generic:Conn_02x01
- added J5: Conn_01x04, Connector_PinHeader_2.54mm:PinHeader_1x04_P2.54mm_Vertical, symbol Connector_Generic:Conn_01x04
- added K1: FINDER-34.51, Relay_THT:Relay_SPDT_Finder_34.51_Vertical, symbol Relay:FINDER-34.51
- added Q1, Q2: IRLZ44N, PCM_Package_TO_SOT_THT_AKL:TO-220-3_Vertical_GDS, symbol PCM_Transistor_MOSFET_AKL:IRLZ44N
- added R1, R2, R3: 47k, Resistor_SMD:R_0201_0603Metric_Pad0.64x0.40mm_HandSolder, symbol Device:R
- U1: value TSR_1-2433 -> TSR_1-2450
Connections:
- net GND: now also U1.2 (GND), C1.1, J3.2 (Pin_2), J5.2 (Pin_2), Q1.3 (S), Q2.3 (S), R1.2, R2.2, R3.1
- net +5V: now reaches ESP32C6.1 (5V)
- net +5V: now also U1.3 (Vout), C1.2
- net +3.3V: now reaches ESP32C6.3 (3.3V)
- net +3.3V: now also J4.1 (Pin_1), J5.1 (Pin_1); no longer U1.3 (Vout)
- net at ESP32C6.4 (GP0): now also Q1.1 (G), R2.1
- net at ESP32C6.5 (GP1): now also Q2.1 (G), R3.2
- net waterlevel_in: now reaches ESP32C6.6 (GP2)
- net waterlevel_in: now also J4.2 (Pin_2), R1.1
- net humidity_scl_i2c: now reaches ESP32C6.7 (GP3)
- net humidity_scl_i2c: now also J5.4 (Pin_4)
- net humidity_sda_i2c: now reaches ESP32C6.8 (GP4)
- net humidity_sda_i2c: now also J5.3 (Pin_3)
- net +9V: now reaches U1.1 (Vin)
- net +9V: now also J2.1 (Pin_1), J3.1 (Pin_1), K1.A2
- new net: J2.2 (Pin_2), Q2.2 (D)
- new net: J1.1 (Pin_1), K1.11
- new net: J1.2 (Pin_2), K1.14
- new net: K1.A1, Q1.2 (D)
- no-connect marks 0 -> 10
Other:
- moved on the sheet: U1
